Commit message: need fix for rotation

File: robosuite/models/assets/robots/dual_kinova3/leonardo.urdf (robot description, URDF)
Before this commit: robot gen3, 11 links, 10 joints
Joints:
- joint base_joint: origin xyz=0 -0.058 0.232548 rpy=-1.5708 0 0 -> xyz=0 0 0 rpy=-1.5708 0 0

Commit message: transoformation matrix issue solved

File: robosuite/models/assets/robots/dual_kinova3/leonardo.urdf (robot description, URDF)
Before this commit: robot gen3, 11 links, 10 joints
Joints:
- joint base_joint: origin xyz=0 0 0 rpy=-1.5708 0 0 -> xyz=0 0 0 rpy=0 0 0
